File: docs/kicad/controller/v_controller.kicad_pcb (KiCad board)
At the start: 2 copper layers, 68.6 x 99.1 mm, 51 parts, among them J1 19.5V, J10 LEFT, J11 RIGHT, J12 MY_DISPLAY_CONN, J13 Sensor Left, J14 Sensor Right, J2 SERVO, J3 5V, J4 GND, J5 WS2812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

Commit message: update CNC3018_ESP and other denormalized kiCad stuff*
Connections:
- J13 pad 1: Net-(J13-Pad1) -> Net-(C1-Pad2)
